File: Board_design/long_board_detector.brd (EAGLE design)
At the start: 103.6 x 43.2 mm, 57 parts, among them IC1 TL072P, IC2 78L05Z, IC3 LM393N, Q1 BC549, Q2 BC549, Q3 BC549, Q4 BC549, X1 22-23-2021, X2 22-23-2021

Commit message: Readme and brd design update
Other:
- board text added: "GRD"
- board text added: "rev 1.1"
- board text removed: "BIDE"
- board text removed: "DGD"
